Commit message: Feat: Front laser sensor

File: ROSpackages/multiple_robot_slam/urdf/robot1.xacro (robot description, xacro)
@@ -1,12 +1,30 @@
 <?xml version='1.0'?>
 <robot name="robot1" xmlns:xacro="http://www.ros.org/wiki/xacro">
-  <material name="darkGreen">
-     <color rgba="0 0 0.4 0"/>
-  </material>
+<!--TODO Change mass (low mass was resulting in strange movement) -->
+  <xacro:include filename="$(find multiple_robot_slam)/urdf/robot1.gazebo" />
+  <link name="robot_footprint"></link>
+  <gazebo reference="chassis">
+    <material>Gazebo/Green</material>
+  </gazebo>
+  <gazebo reference="front_right_wheel">
+    <material>Gazebo/Orange</material>
+  </gazebo>
+  <gazebo reference="front_left_wheel" >
+    <material>Gazebo/Orange</material>
+  </gazebo>
+  <gazebo reference="back_right_wheel">
+    <material>Gazebo/Orange</material>
+  </gazebo>
+  <gazebo reference="back_left_wheel">
+    <material>Gazebo/Orange</material>
+  </gazebo>
+  <gazebo reference="hokuyo">
+    <material>Gazebo/Red</material>
+  </gazebo>
   <link name='chassis'>
     <pose>0 0 0.1 0 0 0</pose>
     <inertial>
       <mass value="2"/>
-      <origin xyz="0.0 0 0" rpy=" 0 0 0"/>
+      <origin xyz="0 0 -0.01" rpy=" 0 0 0"/>
       <inertia
           ixx="0.1" ixy="0" ixz="0"
@@ -15,4 +33,10 @@
       />
     </inertial>
+    <visual name='chassis_visual'>
+      <origin xyz="0 0 0" rpy=" 0 0 0"/>
+      <geometry>
+        <box size=".06 .12 .03"/>
+      </geometry>
+    </visual>
     <collision name='chassis_collision'>
       <origin xyz="0 0 0" rpy=" 0 0 0"/>
@@ -21,105 +45,126 @@
       </geometry>
     </collision>
-    <visual name='chassis_visual'>
-	  <origin xyz="0 0 0" rpy=" 0 0 0"/>
-      <geometry>
-    		<box size=".06 .12 .03"/>
-      </geometry>
-      <material name="darkGreen"/>
-    </visual>
-  </link>
- <!--link name='front_right_wheel_hinge'>
-    <inertial>
-      <mass value="0.5"/>
-      <origin xyz="0.0 0 0" rpy=" 0 0 0"/>
-      <inertia
-          ixx="0.1" ixy="0" ixz="0"
-          iyy="0.1" iyz="0"
-          izz="0.1"
+  </link>
+  <link name='front_right_wheel'>
+    <inertial>
+      <mass value=".1"/>
+      <origin xyz="0.0 0 0" rpy=" 0 0 0"/>
+      <inertia
+          ixx="0.001" ixy="0" ixz="0"
+          iyy="0.001" iyz="0"
+          izz="0.001"
       />
     </inertial>
     <visual name='front_right_wheel_visual'>
-      <origin xyz="0 0 0" rpy=" 0 1.5707 1.5707"/>
-      <geometry>
-        <cylinder radius="0.03" length="0.01"/>
-      </geometry>
+      <origin xyz="0 0 0" rpy=" 0 1.5707 0"/>
+      <geometry>
+        <cylinder radius="0.03" length="0.01"/>
+      </geometry>
+      <material name="darkGreen"/>
     </visual>
     <collision name='front_right_wheel_collision'>
-      <origin xyz="0 0 0" rpy=" 0 1.5707 1.5707"/>
-      <geometry>
-        <cylinder radius="0.03" length="0.01"/>
-      </geometry>
-    </collision>
- </link>
- <link name='front_left_wheel_hinge'>
-    <inertial>
-      <mass value="0.5"/>
-      <origin xyz="0.0 0 0" rpy=" 0 0 0"/>
-      <inertia
-          ixx="0.1" ixy="0" ixz="0"
-          iyy="0.1" iyz="0"
-          izz="0.1"
+      <origin xyz="0 0 0" rpy=" 0 1.5707 0"/>
+      <geometry>
+        <cylinder radius="0.03" length="0.01"/>
+      </geometry>
+    </collision>
+  </link>
+  <link name='front_left_wheel'>
+    <inertial>
+      <mass value=".1"/>
+      <origin xyz="0.0 0 0" rpy=" 0 0 0"/>
+      <inertia
+          ixx="0.001" ixy="0" ixz="0"
+          iyy="0.001" iyz="0"
+          izz="0.001"
       />
     </inertial>
     <visual name='front_left_wheel_visual'>
-      <origin xyz="0 0 0" rpy=" 0 1.5707 1.5707"/>
-      <geometry>
-        <cylinder radius="0.03" length="0.01"/>
-      </geometry>
+      <origin xyz="0 0 0" rpy=" 0 1.5707 0"/>
+      <geometry>
+        <cylinder radius="0.03" length="0.01"/>
+      </geometry>
+      <material name="darkGreen"/>
     </visual>
     <collision name='front_left_wheel_collision'>
-      <origin xyz="0 0 0" rpy=" 0 1.5707 1.5707"/>
-      <geometry>
-        <cylinder radius="0.03" length="0.01"/>
-      </geometry>
-    </collision>
- </link>
- <link name='back_right_wheel_hinge'>
-    <inertial>
-      <mass value="0.5"/>
-      <origin xyz="0.0 0 0" rpy=" 0 0 0"/>
-      <inertia
-          ixx="0.1" ixy="0" ixz="0"
-          iyy="0.1" iyz="0"
-          izz="0.1"
+      <origin xyz="0 0 0" rpy=" 0 1.5707 0"/>
+      <geometry>
+        <cylinder radius="0.03" length="0.01"/>
+      </geometry>
+    </collision>
+  </link>
+  <link name='back_right_wheel'>
+    <inertial>
+      <mass value=".1"/>
+      <origin xyz="0.0 0 0" rpy=" 0 0 0"/>
+      <inertia
+          ixx="0.001" ixy="0" ixz="0"
+          iyy="0.001" iyz="0"
+          izz="0.001"
       />
     </inertial>
     <visual name='back_right_wheel_visual'>
-      <origin xyz="0 0 0" rpy=" 0 1.5707 1.5707"/>
-      <geometry>
-        <cylinder radius="0.03" length="0.01"/>
-      </geometry>
+      <origin xyz="0 0 0" rpy=" 0 1.5707 0"/>
+      <geometry>
+        <cylinder radius="0.03" length="0.01"/>
+      </geometry>
+      <material name="darkGreen"/>
     </visual>
     <collision name='back_right_wheel_collision'>
-      <origin xyz="0 0 0" rpy=" 0 1.5707 1.5707"/>
-      <geometry>
-        <cylinder radius="0.03" length="0.01"/>
-      </geometry>
-    </collision>
- </link>
- <link name='back_left_wheel_hinge'>
-    <inertial>
-      <mass value="0.5"/>
-      <origin xyz="0.0 0 0" rpy=" 0 0 0"/>
-      <inertia
-          ixx="0.1" ixy="0" ixz="0"
-          iyy="0.1" iyz="0"
-          izz="0.1"
+      <origin xyz="0 0 0" rpy=" 0 1.5707 0"/>
+      <geometry>
+        <cylinder radius="0.03" length="0.01"/>
+      </geometry>
+    </collision>
+  </link>
+  <link name='back_left_wheel'>
+    <inertial>
+      <mass value=".1"/>
+      <origin xyz="0.0 0 0" rpy=" 0 0 0"/>
+      <inertia
+          ixx="0.001" ixy="0" ixz="0"
+          iyy="0.001" iyz="0"
+          izz="0.001"
       />
     </inertial>
     <visual name='back_left_wheel_visual'>
-      <origin xyz="0 0 0" rpy=" 0 1.5707 1.5707"/>
-      <geometry>
-        <cylinder radius="0.03" length="0.01"/>
-      </geometry>
+      <origin xyz="0 0 0" rpy=" 0 1.5707 0"/>
+      <geometry>
+        <cylinder radius="0.03" length="0.01"/>
+      </geometry>
+      <material name="darkGreen"/>
     </visual>
     <collision name='back_left_wheel_collision'>
-      <origin xyz="0 0 0" rpy=" 0 1.5707 1.5707"/>
-      <geometry>
-        <cylinder radius="0.03" length="0.01"/>
-      </geometry>
-    </collision>
- </link>
-<!-- Joints ->
+      <origin xyz="0 0 0" rpy=" 0 1.5707 0"/>
+      <geometry>
+        <cylinder radius="0.03" length="0.01"/>
+      </geometry>
+    </collision>
+  </link>
+<!-- Laser Sensor -->
+  <link name='hokuyo'>
+    <inertial>
+      <mass value="1e-5"/>
+      <origin xyz="0 0 0" rpy=" 0 0 0"/>
+      <inertia
+    	  ixx="1e-6" ixy="0" ixz="0"
+    	  iyy="1e-6" iyz="0"
+    	  izz="1e-6"
+      />
+    </inertial>
+    <visual name='laser_visual'>
+      <origin xyz="0 0 0" rpy=" 0 0 0"/>
+      <geometry>
+	        <cylinder radius="0.01" length="0.02"/>
+      </geometry>
+    </visual>
+    <collision name='laser_collision'>
+      <origin xyz="0 0 0" rpy=" 0 0 0"/>
+      <geometry>
+	       <cylinder radius="0.01" length="0.02"/>
+      </geometry>
+    </collision>
+  </link>
+<!-- Joints -->
   <joint name="robot_footprint_joint" type="fixed">
     <origin xyz="0 0 0" rpy="0 0 0" />
@@ -128,34 +173,40 @@
   </joint>
   <joint type="continuous" name="front_right_wheel_hinge">
-    <origin xyz="0.031 0.045 0" rpy="0 0 0"/>
-    <child link="left_wheel"/>
+    <origin xyz="0.035 0.045 0" rpy="0 0 0"/>
+    <child link="front_right_wheel"/>
     <parent link="chassis"/>
-    <axis xyz="0 1 0" rpy="0 0 0"/>
+    <axis xyz="1 0 0" rpy="0 0 0"/>
     <limit effort="10000" velocity="1000"/>
     <dynamics damping="1.0" friction="1.0"/>
    </joint>
   <joint type="continuous" name="front_left_wheel_hinge">
-      <origin xyz="-0.031 0.045 0" rpy="0 0 0"/>
-      <child link="right_wheel"/>
+      <origin xyz="-0.035 0.045 0" rpy="0 0 0"/>
+      <child link="front_left_wheel"/>
       <parent link="chassis"/>
-      <axis xyz="0 1 0" rpy="0 0 0"/>
+      <axis xyz="1 0 0" rpy="0 0 0"/>
       <limit effort="10000" velocity="1000"/>
       <dynamics damping="1.0" friction="1.0"/>
     </joint>
   <joint type="continuous" name="back_right_wheel_hinge">
-      <origin xyz="0.031 -0.045 0" rpy="0 0 0"/>
-      <child link="right_wheel"/>
+      <origin xyz="0.035 -0.045 0" rpy="0 0 0"/>
+      <child link="back_right_wheel"/>
       <parent link="chassis"/>
-      <axis xyz="0 1 0" rpy="0 0 0"/>
+      <axis xyz="1 0 0" rpy="0 0 0"/>
       <limit effort="10000" velocity="1000"/>
       <dynamics damping="1.0" friction="1.0"/>
     </joint>
   <joint type="continuous" name="back_left_wheel_hinge">
-      <origin xyz="-0.031 -0.045 0" rpy="0 0 0"/>
-      <child link="right_wheel"/>
+      <origin xyz="-0.035 -0.045 0" rpy="0 0 0"/>
+      <child link="back_left_wheel"/>
       <parent link="chassis"/>
-      <axis xyz="0 1 0" rpy="0 0 0"/>
+      <axis xyz="1 0 0" rpy="0 0 0"/>
       <limit effort="10000" velocity="1000"/>
       <dynamics damping="1.0" friction="1.0"/>
-    </joint-->
+    </joint>
+<joint type="fixed" name="hokuyo_joint">
+    <origin xyz="0 0.05 0.018" rpy="0 0 1.5707"/>
+    <child link="hokuyo"/>
+    <parent link="chassis"/>
+    <axis xyz="0 1 0" rpy="0 0 0"/>
+</joint>
 </robot>
